File: hardware/industrial-dual-ac-relay.kicad_pcb (KiCad board)
At the start: 2 copper layers, 40 x 40 mm, 29 parts, among them P1 CON-SENSOR, P2 Digital Output, P3 Debug, P4 Boot, U1 XMC1100, U2 AQH3213AX, U5 AQH3213AX, U6 DRILL, U7 DRILL, U8 DRILL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

Commit message: Version V1.1 : Changed pins to highoutput, changed resistor order
Parts:
- C1: value 100nF -> 1uF
- RP4: value 1k -> 10k
- moved P3 3.46 mm to (101.0, 51.0)
- moved R5 1.10 mm to (106.8, 40.5), turned to 270 degrees
- moved D1 1.10 mm to (108.2, 40.5), turned to 270 degrees
- moved C4 0.10 mm to (103.2, 46.9)
Connections:
- RP4 pad 1: Net-(RP1-Pad1) -> OUTPUT0
- RP4 pad 4: Net-(RP1-Pad4) -> OUTPUT1
- U1 pad 11: Net-(U1-Pad11) -> Net-(P4-Pad2)
- U1 pad 12: Net-(P4-Pad2) -> Net-(P3-Pad1)
- U1 pad 13: Net-(P3-Pad1) -> OUTPUT0
- U1 pad 14: OUTPUT0 -> OUTPUT1
- U1 pad 15: OUTPUT1 -> Net-(U1-Pad15)
Routing:
- net OUTPUT0: track 9.76 -> 17.3 mm
- net OUTPUT1: track 12.1 -> 19.0 mm
- net Net-(RP1-Pad1): track 14.8 -> 9.02 mm
- net GND: track 34.5 -> 30.0 mm, vias 13 -> 20
- net 3V3: track 48.5 -> 52.5 mm
- net Net-(P3-Pad1): track 2.11 -> 5.19 mm
- added copper zone on F.Cu, net GND
Other:
- board text added: "Industrial Dual AC Relay 1.1"
- board text removed: "Industrial Dual AC Relay 1.0"
