File: hardware/industrial-dual-ac-relay.kicad_sch (KiCad schematic)
At the start: 25 parts, among them P2 Digital Output

Commit message: Data cleanup
Parts:
- C1: value (none) -> 1uF; footprint (none) -> kicad-libraries:C0603F
- C2: value (none) -> 220pF; footprint (none) -> kicad-libraries:C0402F
- C3: value (none) -> 10uF; footprint (none) -> kicad-libraries:C0805
- C4: value (none) -> 100nF; footprint (none) -> kicad-libraries:C0603F
- D1, D2, D5: value (none) -> blue; footprint (none) -> kicad-libraries:D0603F
- P1: value (none) -> CON-SENSOR; footprint (none) -> kicad-libraries:CON-SENSOR2
- P3: value (none) -> Debug; footprint (none) -> kicad-libraries:DEBUG_PAD
- P4: value (none) -> Boot; footprint (none) -> kicad-libraries:SolderJumper
- R1, R4: value (none) -> MOV-10D391KTR; footprint (none) -> kicad-libraries:VAR_10mm
- R5: value (none) -> 1k; footprint (none) -> kicad-libraries:R0603F
- RP1: value (none) -> 150; footprint (none) -> kicad-libraries:0603X4
- RP2: value (none) -> 82; footprint (none) -> kicad-libraries:4X0402
- RP3: value (none) -> 1k; footprint (none) -> kicad-libraries:0603X4
- RP4: value (none) -> 10k; footprint (none) -> kicad-libraries:0603X4
- U1: value (none) -> XMC1100; footprint (none) -> kicad-libraries:QFN24-4x4mm-0.5mm
- U2, U5: value (none) -> AQH3213AX; footprint (none) -> kicad-libraries:AQ-H
- U6, U7, U8, U9: value (none) -> DRILL; footprint (none) -> kicad-libraries:DRILL_NP_New
Other:
- note added: "Copyright Tinkerforge GmbH 2023. This documentation describes Open Hardware and is licensed under the CERN OHL v. 1.1. You may redistribute and modify this documentation under the terms of the CERN OHL v.1.1. (http://ohwr.org/cernohl). This documentation is distributed WITHOUT ANY EXPRESS OR IMPLIED WARRANTY, INCLUDING OF MERCHANTABILITY, SATISFACTORY QUALITY AND FITNESS FOR A PARTICULAR PURPOSE.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"
- note removed: "Copyright Tinkerforge GmbH 2020. This documentation describes Open Hardware and is licensed under the CERN OHL v. 1.1. You may redistribute and modify this documentation under the terms of the CERN OHL v.1.1. (http://ohwr.org/cernohl). This documentation is distributed WITHOUT ANY EXPRESS OR IMPLIED WARRANTY, INCLUDING OF MERCHANTABILITY, SATISFACTORY QUALITY AND FITNESS FOR A PARTICULAR PURPOSE.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"

Commit message: Data cleanup
Parts:
- U7, U8, U9: footprint kicad-libraries:DRILL_NP_New -> kicad-libraries:DRILL_NP
- Ue1: renamed from U6; footprint kicad-libraries:DRILL_NP_New -> kicad-libraries:DRILL_NP
Changed lines of the file:
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@@
       (effects (font (size 1.524 1.524)))
     )
-    (property "Footprint" "kicad-libraries:DRILL_NP_New" (id 2) (at 279.4 161.29 0)
+    (property "Footprint" "kicad-libraries:DRILL_NP" (id 2) (at 279.4 161.29 0)
       (effects (font (size 1.524 1.524)) hide)
     )
@@
       (effects (font (size 1.524 1.524)))
     )
-    (property "Footprint" "kicad-libraries:DRILL_NP_New" (id 2) (at 279.4 154.94 0)
+    (property "Footprint" "kicad-libraries:DRILL_NP" (id 2) (at 279.4 154.94 0)
       (effects (font (size 1.524 1.524)) hide)
     )
@@
   (symbol (lib_id "tinkerforge:DRILL") (at 270.51 154.94 0) (unit 1)
     (in_bom yes) (on_board yes)
-    (property "Reference" "U6" (id 0) (at 271.78 153.67 0)
+    (property "Reference" "Ue1" (id 0) (at 271.78 153.67 0)
       (effects (font (size 1.524 1.524)) hide)
     )
@@
       (effects (font (size 1.524 1.524)))
     )
-    (property "Footprint" "kicad-libraries:DRILL_NP_New" (id 2) (at 270.51 154.94 0)
+    (property "Footprint" "kicad-libraries:DRILL_NP" (id 2) (at 270.51 154.94 0)
       (effects (font (size 1.524 1.524)) hide)
     )
@@
       (effects (font (size 1.524 1.524)))
     )
-    (property "Footprint" "kicad-libraries:DRILL_NP_New" (id 2) (at 270.51 161.29 0)
+    (property "Footprint" "kicad-libraries:DRILL_NP" (id 2) (at 270.51 161.29 0)
       (effects (font (size 1.524 1.524)) hide)
     )
@@
       (reference "U5") (unit 1) (value "AQH3213AX") (footprint "kicad-libraries:AQ-H")
     )
+    (path "/00000000-0000-0000-0000-00005006691c"
+      (reference "U7") (unit 1) (value "DRILL") (footprint "kicad-libraries:DRILL_NP")
+    )
+    (path "/00000000-0000-0000-0000-000050066918"
+      (reference "U8") (unit 1) (value "DRILL") (footprint "kicad-libraries:DRILL_NP")
+    )
+    (path "/00000000-0000-0000-0000-000050066905"
+      (reference "U9") (unit 1) (value "DRILL") (footprint "kicad-libraries:DRILL_NP")
+    )
     (path "/00000000-0000-0000-0000-00005006691a"
-      (reference "U6") (unit 1) (value "DRILL") (footprint "kicad-libraries:DRILL_NP_New")
-    )
-    (path "/00000000-0000-0000-0000-00005006691c"
-      (reference "U7") (unit 1) (value "DRILL") (footprint "kicad-libraries:DRILL_NP_New")
-    )
-    (path "/00000000-0000-0000-0000-000050066918"
-      (reference "U8") (unit 1) (value "DRILL") (footprint "kicad-libraries:DRILL_NP_New")
-    )
-    (path "/00000000-0000-0000-0000-000050066905"
-      (reference "U9") (unit 1) (value "DRILL") (footprint "kicad-libraries:DRILL_NP_New")
-    )
-  )
+      (reference "Ue1") (unit 1) (value "DRILL") (footprint "kicad-libraries:DRILL_NP")
+    )
+  )
